File: battery_pack_usb.kicad_sch (KiCad schematic)
At the start: 25 parts, among them J1 Conn_01x02_Male, J2 USB_C_Receptacle_USB2.0, SW1 SW_SPST, U1 BQ25886

Commit message: Improve circuit and PCB
Parts:
- removed SW1: SW_SPST, Connector_PinHeader_2.00mm:PinHeader_1x02_P2.00mm_Vertical, symbol Switch:SW_SPST
- added D3: Green, Connector_Molex:Molex_PicoBlade_53047-0210_1x02_P1.25mm_Vertical, symbol Device:LED
- added D4, D5, D6: ESD5Zxx, Diode_SMD:D_SOD-523, symbol Diode:ESD5Zxx
- added H1, H2: MountingHole, MountingHole:MountingHole_3.2mm_M3_ISO14580, symbol Mechanical:MountingHole
- added R10, R9: 5k1, Resistor_SMD:R_0603_1608Metric_Pad0.98x0.95mm_HandSolder, symbol Device:R
- BT1: footprint Connector_PinHeader_2.54mm:PinHeader_1x02_P2.54mm_Vertical -> Connector_Molex:Molex_PicoBlade_53047-0210_1x02_P1.25mm_Vertical
- C1: value 1u 5V -> 1u; footprint Capacitor_SMD:C_0603_1608Metric_Pad1.05x0.95mm_HandSolder -> Capacitor_SMD:C_0603_1608Metric_Pad1.08x0.95mm_HandSolder
- C2, C3: value 10u 5V -> 10u; footprint Capacitor_SMD:C_0805_2012Metric -> Capacitor_SMD:C_0805_2012Metric_Pad1.18x1.45mm_HandSolder
- C4, C5: footprint Capacitor_SMD:C_0603_1608Metric_Pad1.05x0.95mm_HandSolder -> Capacitor_SMD:C_0603_1608Metric_Pad1.08x0.95mm_HandSolder
- C6: value 10u 9V -> 10u 10V; footprint Capacitor_SMD:C_0805_2012Metric -> Capacitor_SMD:C_0805_2012Metric_Pad1.18x1.45mm_HandSolder
- C7, C8: value 22u 9V -> 22u 10V; footprint Capacitor_SMD:C_0805_2012Metric -> Capacitor_SMD:C_0805_2012Metric_Pad1.18x1.45mm_HandSolder
- D1: value LED -> Red; footprint LED_SMD:LED_0603_1608Metric_Pad1.05x0.95mm_HandSolder -> Connector_Molex:Molex_PicoBlade_53047-0210_1x02_P1.25mm_Vertical
- D2: value LED -> Blue
- J1: value Conn_01x02_Male -> Output; footprint Connector_PinHeader_2.54mm:PinHeader_1x02_P2.54mm_Vertical -> Connector_Molex:Molex_PicoBlade_53047-0210_1x02_P1.25mm_Vertical
- J2: value USB_C_Receptacle_USB2.0 -> USB_C_Receptacle_USB2.0_16P; symbol Connector:USB_C_Receptacle_USB2.0 -> Connector:USB_C_Receptacle_USB2.0_16P
- L1: value 1u -> 1u (XGL3515-102); footprint Inductor_SMD:L_1008_2520Metric -> extraFootprints:XxL3515; Name DFE252012F-1R0M=P2 -> (none)
- R1, R2, R3, R4, R6, R8: footprint Resistor_SMD:R_0603_1608Metric_Pad1.05x0.95mm_HandSolder -> Resistor_SMD:R_0603_1608Metric_Pad0.98x0.95mm_HandSolder
- R5: value 7k5 -> 4k7; footprint Resistor_SMD:R_0603_1608Metric_Pad1.05x0.95mm_HandSolder -> Resistor_SMD:R_0603_1608Metric_Pad0.98x0.95mm_HandSolder
- R7: value 10k -> R; footprint Resistor_SMD:R_0603_1608Metric_Pad1.05x0.95mm_HandSolder -> Resistor_SMD:R_0603_1608Metric_Pad0.98x0.95mm_HandSolder
- TH1: footprint Connector_PinHeader_2.00mm:PinHeader_1x02_P2.00mm_Vertical -> Connector_Molex:Molex_PicoBlade_53047-0210_1x02_P1.25mm_Vertical
Connections:
- net D+: now also D5.1 (K)
- net D-: now also D6.1 (K)
- net GND: now also C1.2, C2.2, U1.5 (OTG), D3.1 (K), D4.2 (A), D5.2 (A), D6.2 (A), R10.2, R9.2; no longer C1.1, C2.1, R7.2
- net REGN: no longer D1.2 (A)
- net at U1.2 (STAT): now also R1.1, R7.1; no longer R1.2
- net V_{Bus}: now reaches J2.A4 (VBUS), J2.A9 (VBUS), J2.B4 (VBUS), J2.B9 (VBUS), U1.23 (VBUS)
- net V_{Bus}: now also C1.1, C2.1, D1.2 (A), D4.1 (K); no longer C1.2, C2.2
- net at J2.A5 (CC1): now also R10.1
- net at J2.B5 (CC2): now also R9.1
- net at D1.1 (K): now also R1.2; no longer R1.1
- net SYS: no longer names the net of C7.1, C8.1, J1.1 (Pin_1), U1.15 (SYS), U1.16 (SYS)
- new net: D3.2 (A), R7.2
- no-connect marks 4 -> 2
Other:
- note added: "2S boost converter - battery charger"
- note added: "R_{ICHGSET} = I_{ICHGSET} * K_{ICHGSET} = I * 3810 mit 4,7k -> 1,23A"
- note added: "USB-C connector"
- note added: "connection to system"
- note added: "mounting holes"
- title: (none) -> 2S USB-C charger v2
- moved on the sheet: BT1, C1, C2, C3, C4, C5, C6, C7, C8, D2, J1, J2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
